File: Electronic/bioreactor.kicad_sch (KiCad schematic)
At the start: 10 parts, among them J1 Conn_01x04_Pin

Commit message: final commit
Parts:
- added C3: 100uF, symbol Device:C
- C1: value C -> 33uF
- C2: value C -> 1uF
Connections:
- net +12V: now also C3.1
- net GND: now also C3.2
Changed lines of the file:
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@@
   (junction (at 58.42 91.44) (diameter 0) (color 0 0 0 0)
   )
+  (junction (at 163.83 64.77) (diameter 0) (color 0 0 0 0)
+  )
   (wire (pts (xy 73.66 71.12) (xy 74.93 71.12))
     (stroke (width 0) (type default))
@@
     (stroke (width 0) (type default))
   )
+  (wire (pts (xy 163.83 62.23) (xy 163.83 64.77))
+    (stroke (width 0) (type default))
+  )
   (wire (pts (xy 128.27 43.18) (xy 128.27 46.99))
     (stroke (width 0) (type default))
@@
     (stroke (width 0) (type default))
   )
+  (wire (pts (xy 168.91 64.77) (xy 163.83 64.77))
+    (stroke (width 0) (type default))
+  )
   (wire (pts (xy 129.54 81.28) (xy 140.97 81.28))
     (stroke (width 0) (type default))
@@
     (stroke (width 0) (type default))
   )
+  (wire (pts (xy 179.07 64.77) (xy 176.53 64.77))
+    (stroke (width 0) (type default))
+  )
   (wire (pts (xy 58.42 99.06) (xy 73.66 99.06))
     (stroke (width 0) (type default))
@@
     (stroke (width 0) (type default))
   )
+  (wire (pts (xy 163.83 64.77) (xy 163.83 68.58))
+    (stroke (width 0) (type default))
+  )
   (symbol (lib_id "power:NEUT") (at 74.93 71.12 270) (unit 1)
     (in_bom yes) (on_board yes) (dnp no) (fields_autoplaced)
@@
         (path "/9da5e5bf-cb24-4e0c-ba6b-22fe9cec6227"
           (reference "#PWR013") (unit 1)
+        )
+      )
+    )
+  )
+  (symbol (lib_id "Device:C") (at 172.72 64.77 90) (unit 1)
+    (in_bom yes) (on_board yes) (dnp no) (fields_autoplaced)
+    (property "Reference" "C3" (at 172.72 58.42 90)
+      (effects (font (size 1.27 1.27)))
+    )
+    (property "Value" "100uF" (at 172.72 60.96 90)
+      (effects (font (size 1.27 1.27)))
+    )
+    (property "Footprint" "" (at 176.53 63.8048 0)
+      (effects (font (size 1.27 1.27)) hide)
+    )
+    (property "Datasheet" "~" (at 172.72 64.77 0)
+      (effects (font (size 1.27 1.27)) hide)
+    )
+    (pin "1")
+    (pin "2")
+    (instances
+      (project "bioreactor"
+        (path "/9da5e5bf-cb24-4e0c-ba6b-22fe9cec6227"
+          (reference "C3") (unit 1)
         )
       )
@@
     )
   )
+  (symbol (lib_id "power:GND") (at 179.07 64.77 90) (unit 1)
+    (in_bom yes) (on_board yes) (dnp no) (fields_autoplaced)
+    (property "Reference" "#PWR019" (at 185.42 64.77 0)
+      (effects (font (size 1.27 1.27)) hide)
+    )
+    (property "Value" "GND" (at 182.88 65.405 90)
+      (effects (font (size 1.27 1.27)) (justify right))
+    )
+    (property "Footprint" "" (at 179.07 64.77 0)
+      (effects (font (size 1.27 1.27)) hide)
+    )
+    (property "Datasheet" "" (at 179.07 64.77 0)
+      (effects (font (size 1.27 1.27)) hide)
+    )
+    (pin "1")
+    (instances
+      (project "bioreactor"
+        (path "/9da5e5bf-cb24-4e0c-ba6b-22fe9cec6227"
+          (reference "#PWR019") (unit 1)
+        )
+      )
+    )
+  )
   (symbol (lib_id "Device:Lamp") (at 128.27 38.1 180) (unit 1)
     (in_bom yes) (on_board yes) (dnp no) (fields_autoplaced)
@@
     )
   )
-  (symbol (lib_id "power:+12V") (at 163.83 68.58 0) (unit 1)
+  (symbol (lib_id "power:+12V") (at 163.83 62.23 0) (unit 1)
     (in_bom yes) (on_board yes) (dnp no)
-    (property "Reference" "#PWR05" (at 163.83 72.39 0)
-      (effects (font (size 1.27 1.27)) hide)
-    )
-    (property "Value" "+12V" (at 163.83 64.77 0)
-      (effects (font (size 1.27 1.27)))
-    )
-    (property "Footprint" "" (at 163.83 68.58 0)
-      (effects (font (size 1.27 1.27)) hide)
-    )
-    (property "Datasheet" "" (at 163.83 68.58 0)
+    (property "Reference" "#PWR05" (at 163.83 66.04 0)
+      (effects (font (size 1.27 1.27)) hide)
+    )
+    (property "Value" "+12V" (at 163.83 58.42 0)
+      (effects (font (size 1.27 1.27)))
+    )
+    (property "Footprint" "" (at 163.83 62.23 0)
+      (effects (font (size 1.27 1.27)) hide)
+    )
+    (property "Datasheet" "" (at 163.83 62.23 0)
       (effects (font (size 1.27 1.27)) hide)
     )
@@
       (effects (font (size 1.27 1.27)) (justify left))
     )
-    (property "Value" "C" (at 93.98 97.155 0)
+    (property "Value" "33uF" (at 93.98 97.155 0)
       (effects (font (size 1.27 1.27)) (justify left))
     )
@@
       (effects (font (size 1.27 1.27)) (justify left))
     )
-    (property "Value" "C" (at 62.23 97.155 0)
-      (effects (font (size 1.27 1.27)) (justify left))
-    )
+    (property "Value" "1uF" (at 62.23 97.155 0)
+      (effects (font (size 1.27 1.27)) (justify left))
+    )
